File: KiCad files/Buggly SPD.kicad_pcb (KiCad board)
At the start: 2 copper layers, 120.4 x 100.1 mm, 87 parts, among them IC1 Trig Cond Socket, J1 Conn_01x07, J2 Conn_01x05, J3 Conn_01x08, J4 Conn_01x02, J5 Conn_02x03_Odd_Even, J6 Conn_01x02, J7 DB25_Male, J8 12V Test, Q1 2N3906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

Commit message: Add files via upload
Parts:
- added C19: .01uf, Capacitor_THT:C_Disc_D5.0mm_W2.5mm_P2.50mm, F.Cu at (154.7, 54.6)
- added R24: 100K, Resistor_THT:R_Axial_DIN0207_L6.3mm_D2.5mm_P7.62mm_Horizontal, F.Cu at (94.0, 83.4)
- added R25: 100K, Resistor_THT:R_Axial_DIN0207_L6.3mm_D2.5mm_P7.62mm_Horizontal, F.Cu at (100.2, 75.8)
- added R26: 100K, Resistor_THT:R_Axial_DIN0207_L6.3mm_D2.5mm_P7.62mm_Horizontal, F.Cu at (93.0, 45.0)
- added R27: 100K, Resistor_THT:R_Axial_DIN0207_L6.3mm_D2.5mm_P7.62mm_Horizontal, F.Cu at (100.6, 51.2)
- added R28: 100K, Resistor_THT:R_Axial_DIN0207_L6.3mm_D2.5mm_P7.62mm_Horizontal, F.Cu at (123.7, 45.1)
- added R29: 100K, Resistor_THT:R_Axial_DIN0207_L6.3mm_D2.5mm_P7.62mm_Horizontal, F.Cu at (131.3, 51.3)
- added R30: 1K, Resistor_THT:R_Axial_DIN0207_L6.3mm_D2.5mm_P7.62mm_Horizontal, F.Cu at (97.1, 75.8)
- added R31: 1K, Resistor_THT:R_Axial_DIN0207_L6.3mm_D2.5mm_P7.62mm_Horizontal, F.Cu at (103.3, 75.8)
- added R32: 1K, Resistor_THT:R_Axial_DIN0207_L6.3mm_D2.5mm_P7.62mm_Horizontal, F.Cu at (131.3, 48.2)
- added R33: 1K, Resistor_THT:R_Axial_DIN0207_L6.3mm_D2.5mm_P7.62mm_Horizontal, F.Cu at (131.3, 54.5)
- added R34: 1K, Resistor_THT:R_Axial_DIN0207_L6.3mm_D2.5mm_P7.62mm_Horizontal, F.Cu at (100.6, 48.1)
- added R35: 1K, Resistor_THT:R_Axial_DIN0207_L6.3mm_D2.5mm_P7.62mm_Horizontal, F.Cu at (100.6, 54.3)
- C18, C20: value 0.1uF -> 1uF
- C21: value 0.1uF -> .01uF
- moved U4 33.6 mm to (102.9, 45.0), turned to 0 degrees
- moved R20 29.3 mm to (102.1, 60.0)
- moved U5 29.3 mm to (94.1, 73.5)
- moved R21 29.3 mm to (94.6, 63.1)
- moved C21 29.0 mm to (154.8, 48.2), turned to 0 degrees
- moved R15 26.7 mm to (116.1, 52.7), turned to 90 degrees
- moved C20 21.1 mm to (154.7, 57.8), turned to 0 degrees
- moved R16 21.0 mm to (113.1, 45.0), turned to 270 degrees
- moved U3 19.9 mm to (133.5, 45.1), turned to 0 degrees
- moved R13 12.4 mm to (146.9, 52.8), turned to 90 degrees
- moved D4 10.8 mm to (152.8, 133.8), turned to 180 degrees
- moved D2 10.6 mm to (158.6, 124.2), turned to 0 degrees
- moved D1 10.5 mm to (135.7, 130.5), turned to 180 degrees
- moved D3 10.3 mm to (91.8, 118.0), turned to 0 degrees
- moved D11 10.2 mm to (161.2, 98.8), turned to 0 degrees
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Connections:
- C18 pad 2: VDD -> 12V
- C21 pad 2: VDD -> 12V
- D1 pad 1: SigRtn -> ADC-Clamp-3
- D1 pad 2: ADC-Clamp-3 -> SigRtn
- D10 pad 1: SigRtn -> ADC-Clamp-7
- D10 pad 2: ADC-Clamp-7 -> SigRtn
- D11 pad 1: GND -> MCU-D19
- D11 pad 2: MCU-D19 -> GND
- D2 pad 1: SigRtn -> ADC-Clamp-5
- D2 pad 2: ADC-Clamp-5 -> SigRtn
- D3 pad 1: SigRtn -> ADC-Clamp-2
- D3 pad 2: ADC-Clamp-2 -> SigRtn
- D4 pad 1: SigRtn -> ADC-Clamp-4
- D4 pad 2: ADC-Clamp-4 -> SigRtn
- D9 pad 1: SigRtn -> ADC-Clamp-6
- D9 pad 2: ADC-Clamp-6 -> SigRtn
- U3 pad 2: MCU-D8 -> Net-(R32-Pad1)
- U3 pad 4: MCU-D9 -> Net-(R33-Pad1)
- U3 pad 6: VDD -> 12V
- U4 pad 2: MCU-D10 -> Net-(R34-Pad1)
- U4 pad 4: MCU-D11 -> Net-(R35-Pad1)
- U4 pad 6: VDD -> 12V
- U5 pad 2: MCU-D52 -> Net-(R30-Pad1)
- U5 pad 4: MCU-D53 -> Net-(R31-Pad1)
Routing:
- net 12V: track 223.9 -> 313.6 mm
- net MCU-D10: track 14.8 -> 46.3 mm
- net MCU-D9: track 36.2 -> 16.0 mm
- net D11-control: track 109.3 -> 125.4 mm, vias 3 -> 1
- net D53-control: track 127.8 -> 143.6 mm, vias 3 -> 2
- net D10-control: track 107.0 -> 122.2 mm, vias 1 -> 3
- net SigRtn: track 522.5 -> 508.7 mm
- net MCU-D11: track 25.7 -> 37.9 mm
- net D52-control: track 124.4 -> 134.7 mm, vias 3 -> 1
- net ADC-Clamp-3: track 35.8 -> 43.6 mm
- net VDD: track 242.3 -> 248.4 mm, vias 1 -> 2
- net ADC-Clamp-4: track 23.8 -> 27.7 mm
- net Net-(R33-Pad1): track 0.00 -> 2.95 mm
- net Net-(R35-Pad1): track 0.00 -> 2.94 mm
- net Net-(R31-Pad1): track 0.00 -> 2.92 mm
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
Commit message: Add files via upload
Parts:
- removed the C3 at (199.9, 133.6)
- added C5: 0.22uF, Capacitor_THT:C_Disc_D5.0mm_W2.5mm_P2.50mm, F.Cu at (176.4, 133.6)
- added J10: Conn_01x02, Connector_PinHeader_2.54mm:PinHeader_1x02_P2.54mm_Vertical, F.Cu at (182.6, 86.6)
- added J11: Conn_01x01, Connector_PinHeader_2.54mm:PinHeader_1x01_P2.54mm_Vertical, F.Cu at (185.1, 94.2)
- added J12: Conn_01x01, Connector_PinHeader_2.54mm:PinHeader_1x01_P2.54mm_Vertical, F.Cu at (185.1, 99.3)
- added J13: Conn_01x02, Connector_PinHeader_2.54mm:PinHeader_1x02_P2.54mm_Vertical, F.Cu at (182.6, 106.9)
- added J7: Conn_01x01, Connector_PinHeader_2.54mm:PinHeader_1x01_P2.54mm_Vertical, F.Cu at (169.9, 63.7)
- added J8: Conn_01x01, Connector_PinHeader_2.54mm:PinHeader_1x01_P2.54mm_Vertical, F.Cu at (162.3, 112.0)
- added J9: Conn_01x02, Connector_PinHeader_2.54mm:PinHeader_1x02_P2.54mm_Vertical, F.Cu at (182.6, 63.7)
- J1: value Conn_01x07 -> Conn_01x01; footprint Connector_PinHeader_2.54mm:PinHeader_1x07_P2.54mm_Vertical -> Connector_PinHeader_2.54mm:PinHeader_1x01_P2.54mm_Vertical
- J2: value Conn_01x05 -> Conn_01x01; footprint Connector_PinHeader_2.54mm:PinHeader_1x05_P2.54mm_Vertical -> Connector_PinHeader_2.54mm:PinHeader_1x01_P2.54mm_Vertical
- J3: value Conn_01x08 -> Conn_01x02; footprint Connector_PinHeader_2.54mm:PinHeader_1x08_P2.54mm_Vertical -> Connector_PinHeader_2.54mm:PinHeader_1x02_P2.54mm_Vertical
- J4: value Conn_01x02 -> Conn_01x03; footprint Connector_PinHeader_2.54mm:PinHeader_1x02_P2.54mm_Vertical -> Connector_PinHeader_2.54mm:PinHeader_1x03_P2.54mm_Vertical
- J5: value Conn_02x03_Odd_Even -> Conn_01x02; footprint Connector_PinHeader_2.54mm:PinHeader_2x03_P2.54mm_Vertical -> Connector_PinHeader_2.54mm:PinHeader_1x02_P2.54mm_Vertical
- J6: value Conn_01x02 -> Conn_01x07; footprint Connector_PinHeader_2.54mm:PinHeader_1x02_P2.54mm_Vertical -> Connector_PinHeader_2.54mm:PinHeader_1x07_P2.54mm_Vertical
- R16: value 22R -> 100K
- R27: value 100K -> 1K
- R35: value 1K -> 22R
- U1, U2: footprint MPXH61115AC6U Adapter:MPXH6115_Adapter_Vertical -> Buggly SPD:MPXH6115_Adapter_Vertical
- moved D7 66.8 mm to (158.4, 127.3)
- moved D3 66.8 mm to (158.4, 124.1)
- moved J6 64.8 mm to (139.4, 112.0)
- moved J4 63.1 mm to (126.7, 112.0)
- moved D4 62.8 mm to (92.0, 118.1), turned to 0 degrees
- moved D8 61.5 mm to (92.0, 121.4), turned to 0 degrees
- moved J5 59.5 mm to (136.9, 63.7), turned to 90 degrees
- moved J3 49.7 mm to (127.7, 63.7)
- moved C17 24.5 mm to (155.3, 90.1)
- moved D11 24.5 mm to (144.1, 81.2)
- moved D14 24.5 mm to (144.1, 84.5)
- moved IC1 24.5 mm to (144.4, 95.4)
- moved R3 21.1 mm to (176.6, 130.4)
- moved U6 20.9 mm to (158.0, 103.1)
- moved C3 18.6 mm to (184.5, 133.6), turned to 180 degrees
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- renumbered J7 to J15
Connections:
- net D10-control renamed D6-control
- net D50-control renamed D45-control
- net D51-control renamed D49-control
- net D52-control renamed D40-control
- net D53-control renamed D38-control
- C14 pad 1: ADC-Clamp-3 -> ADC-Clamp-0
- C15 pad 1: ADC-Clamp-4 -> ADC-Clamp-1
- C16 pad 1: ADC-Clamp-5 -> ADC-Clamp-2
- C6 pad 1: ADC-Clamp-2 -> ADC-Clamp-4
- C7 pad 1: MCU-A1 -> MCU-A3
- C8 pad 1: MCU-A0 -> MCU-A5
- D1 pad 1: ADC-Clamp-3 -> ADC-Clamp-0
- D10 pad 1: ADC-Clamp-7 -> ADC-Clamp-6
- D12 pad 1: ADC-Clamp-6 -> ADC-Clamp-8
- D13 pad 1: ADC-Clamp-7 -> ADC-Clamp-6
- D2 pad 1: ADC-Clamp-5 -> ADC-Clamp-1
- D5 pad 1: ADC-Clamp-3 -> ADC-Clamp-0
- D6 pad 1: ADC-Clamp-5 -> ADC-Clamp-1
- D9 pad 1: ADC-Clamp-6 -> ADC-Clamp-8
- J15 pad 6: D11-control -> D5-control
- J3 pad 1: MCU-A0 -> MCU-D9
- J3 pad 2: MCU-A1 -> MCU-D8
- J4 pad 1: Net-(J4-Pad1) -> VDD
- J4 pad 2: MCU-D19 -> GND
- J5 pad 1: MCU-D50 -> MCU-D6
- J5 pad 2: MCU-D51 -> MCU-D5
- J6 pad 1: VDD -> ADC-Clamp-0
- J6 pad 2: VDD -> ADC-Clamp-1
- R10 pad 1: ADC-Clamp-3 -> ADC-Clamp-0
- R11 pad 1: ADC-Clamp-4 -> ADC-Clamp-1
- R12 pad 1: ADC-Clamp-5 -> ADC-Clamp-2
- R16 pad 1: D11-control -> GND
- R16 pad 2: Net-(R16-Pad2) -> MCU-D5
- R24 pad 1: MCU-D52 -> MCU-D40
- R25 pad 2: MCU-D53 -> MCU-D38
- R26 pad 1: MCU-D10 -> MCU-D6
- R27 pad 1: GND -> Net-(R27-Pad1)
- R27 pad 2: MCU-D11 -> MCU-D5
- R3 pad 1: ADC-Clamp-7 -> ADC-Clamp-8
- R30 pad 2: MCU-D52 -> MCU-D40
- R31 pad 2: MCU-D53 -> MCU-D38
- R34 pad 2: MCU-D10 -> MCU-D6
- R35 pad 1: Net-(R35-Pad1) -> D5-control
- R35 pad 2: MCU-D11 -> Net-(R35-Pad2)
- R4 pad 1: ADC-Clamp-2 -> ADC-Clamp-4
- R5 pad 1: MCU-A1 -> MCU-A3
- R6 pad 1: MCU-A0 -> MCU-A5
- U4 pad 4: Net-(R35-Pad1) -> Net-(R27-Pad1)
- U4 pad 5: Net-(R16-Pad2) -> Net-(R35-Pad2)
- U6 pad 6: MCU-D50 -> MCU-D45
- U6 pad 7: MCU-D51 -> MCU-D49
Routing:
- net MCU-D52: track 132.0 -> 0.00 mm, vias 1 -> 0
- net MCU-D53: track 130.0 -> 0.00 mm
- net D11-control: track 125.4 -> 0.00 mm, vias 1 -> 0
- net D5-control: track 0.00 -> 123.1 mm, vias 0 -> 3
- net MCU-D40: track 0.00 -> 114.2 mm, vias 0 -> 1
- net MCU-D38: track 0.00 -> 107.8 mm
- net ADC-Clamp-7: track 60.4 -> 0.00 mm
- net MCU-D6: track 0.00 -> 57.6 mm, vias 0 -> 1
- net MCU-D5: track 0.00 -> 54.9 mm
- net SigRtn: track 508.7 -> 454.3 mm, vias 7 -> 4
- net ADC-Clamp-4: track 27.7 -> 79.8 mm, vias 0 -> 2
- net MCU-A3: track 0.00 -> 51.3 mm
- net MCU-A5: track 0.00 -> 51.3 mm, vias 0 -> 1
- net MCU-D51: track 49.1 -> 0.00 mm, vias 1 -> 0
- net MCU-D10: track 46.3 -> 0.00 mm
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Other:
- board text added: "38"
- board text added: "40"
- board text added: "45"
- board text added: "49"
- board text added: "5"
- board text added: "6"
- board text added: "A8"
- board text added: "PWM Idle& Spare"
- board text removed: "10"
- board text removed: "11"
- board text removed: "12"
- board text removed: "13"
- board text removed: "18"
- board text removed: "50"
- board text removed: "51"
- board text removed: "52"
- board text removed: "53"
- board text removed: "A7"
- board text removed: "Idle&Spare"
- board text removed: "N/C"
- board text removed: "Spare"

Commit message: Add files via upload
Parts:
- removed D1, D10, D11, D2, D3, D4, D9: 1N5231B, Diode_THT:D_DO-41_SOD81_P10.16mm_Horizontal
- removed D12, D13, D14, D5, D6, D7, D8: 1N5818, Diode_THT:D_DO-41_SOD81_P10.16mm_Horizontal
- added J16: SP721APP, Package_DIP:DIP-8_W7.62mm, F.Cu at (130.5, 94.9)
- added J17: Conn_01x02, Connector_PinHeader_2.54mm:PinHeader_1x02_P2.54mm_Vertical, F.Cu at (149.6, 63.7)
- added J18: Conn_01x04, Connector_PinSocket_2.54mm:PinSocket_1x04_P2.54mm_Horizontal, F.Cu at (91.3, 59.7)
- added R36: 1K, Resistor_THT:R_Axial_DIN0207_L6.3mm_D2.5mm_P7.62mm_Horizontal, F.Cu at (94.5, 70.9)
- added R37: 2.2K, Resistor_THT:R_Axial_DIN0207_L6.3mm_D2.5mm_P7.62mm_Horizontal, F.Cu at (91.3, 78.5)
- moved C13 13.4 mm to (182.3, 127.4)
- moved C9 13.4 mm to (190.3, 127.4)
- moved R9 13.4 mm to (182.4, 124.3)
- moved C3 9.60 mm to (177.2, 127.3)
- moved C5 9.60 mm to (169.1, 127.4)
- moved R3 9.60 mm to (169.3, 124.2)
- moved R20 7.47 mm to (109.6, 60.0)
- moved R24 7.47 mm to (101.5, 83.4)
- moved R31 7.47 mm to (110.8, 75.8)
- moved U5 7.47 mm to (101.6, 73.5)
- moved R21 7.47 mm to (102.0, 63.1)
- moved R25 7.47 mm to (107.7, 75.8)
- moved R30 7.47 mm to (104.6, 75.8)
- moved C12 7.26 mm to (164.2, 127.3)
- moved C16 7.26 mm to (156.0, 127.3)
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Routing:
- net MCU-D0: track 0.00 -> 83.7 mm, vias 0 -> 3
- net MCU-D1: track 0.00 -> 69.4 mm, vias 0 -> 2
- net SigRtn: track 454.3 -> 407.0 mm
- net VDD: track 288.4 -> 318.8 mm
- net ADC-Clamp-8: track 33.8 -> 60.0 mm
- net ADC-Clamp-2: track 34.7 -> 59.6 mm
- net ADC-Clamp-4: track 79.8 -> 102.8 mm
- net ADC-Clamp-6: track 55.7 -> 76.9 mm
- net ADC-Clamp-1: track 24.4 -> 45.3 mm
- net ADC-Clamp-0: track 37.6 -> 51.6 mm
- net VDDA: track 275.0 -> 285.0 mm, vias 4 -> 6
- net MCU-D38: track 107.8 -> 98.9 mm
- net MCU-D40: track 114.2 -> 105.4 mm
- net D38-control: track 142.8 -> 134.8 mm
- net Spare-ADC: track 69.4 -> 62.4 mm
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Other:
- board text added: "0"
- board text added: "1"
- board text added: "BT RX"
- board text added: "BT TX"
- board text added: "Spare"
