File: KiCad files/file638ED684.sch (KiCad schematic (older format))
At the start: 46 parts, among them IC1 Trig Cond Socket, U1 MPXH6115_Adapter_Vertical, U2 MPXH6115_Adapter_Vertical

Commit message: Add files via upload
Other:
- moved on the sheet: D10, D12, D13, D2, D3, D6, D7, D9
Changed lines of the file:
@@
 L Diode:1N5818 D13
 U 1 1 63914F03
-P 10200 2750
-F 0 "D13" H 10200 2967 50  0000 C CNN
-F 1 "1N5818" H 10200 2876 50  0000 C CNN
-F 2 "Diode_THT:D_DO-41_SOD81_P10.16mm_Horizontal" H 10200 2575 50  0001 C CNN
-F 3 "http://www.vishay.com/docs/88525/1n5817.pdf" H 10200 2750 50  0001 C CNN
-	1    10200 2750
-	1    0    0    -1
-$EndComp
-Wire Wire Line
-	10350 2750 10450 2750
-Wire Wire Line
-	10050 2750 9950 2750
-Wire Wire Line
-	9950 2750 9950 2850
-Wire Wire Line
-	9950 2950 10050 2950
-Text GLabel 9800 2850 0    50   Input ~ 0
+P 10200 2950
+F 0 "D13" H 10200 3167 50  0000 C CNN
+F 1 "1N5818" H 10200 3076 50  0000 C CNN
+F 2 "Diode_THT:D_DO-41_SOD81_P10.16mm_Horizontal" H 10200 2775 50  0001 C CNN
+F 3 "http://www.vishay.com/docs/88525/1n5817.pdf" H 10200 2950 50  0001 C CNN
+	1    10200 2950
+	1    0    0    -1
+$EndComp
+Wire Wire Line
+	10350 2950 10450 2950
+Wire Wire Line
+	10050 2950 9950 2950
+Wire Wire Line
+	9950 2950 9950 3050
+Wire Wire Line
+	9950 3150 10050 3150
+Text GLabel 9800 3050 0    50   Input ~ 0
 ADC-Clamp-7
 Wire Wire Line
-	9800 2850 9950 2850
-Connection ~ 9950 2850
-Wire Wire Line
-	9950 2850 9950 2950
+	9800 3050 9950 3050
+Connection ~ 9950 3050
+Wire Wire Line
+	9950 3050 9950 3150
 $Comp
 L Device:C C2
@@
 L Diode:1N5818 D6
 U 1 1 63914F48
-P 8250 1900
-F 0 "D6" H 8250 2117 50  0000 C CNN
-F 1 "1N5818" H 8250 2026 50  0000 C CNN
-F 2 "Diode_THT:D_DO-41_SOD81_P10.16mm_Horizontal" H 8250 1725 50  0001 C CNN
-F 3 "http://www.vishay.com/docs/88525/1n5817.pdf" H 8250 1900 50  0001 C CNN
-	1    8250 1900
-	1    0    0    -1
-$EndComp
-Wire Wire Line
-	8400 1900 8500 1900
-Wire Wire Line
-	8100 1900 8000 1900
-Wire Wire Line
-	8000 1900 8000 2000
-Wire Wire Line
-	8000 2100 8100 2100
-Text GLabel 7850 2000 0    50   Input ~ 0
+P 8250 2000
+F 0 "D6" H 8250 2217 50  0000 C CNN
+F 1 "1N5818" H 8250 2126 50  0000 C CNN
+F 2 "Diode_THT:D_DO-41_SOD81_P10.16mm_Horizontal" H 8250 1825 50  0001 C CNN
+F 3 "http://www.vishay.com/docs/88525/1n5817.pdf" H 8250 2000 50  0001 C CNN
+	1    8250 2000
+	1    0    0    -1
+$EndComp
+Wire Wire Line
+	8400 2000 8500 2000
+Wire Wire Line
+	8100 2000 8000 2000
+Wire Wire Line
+	8000 2000 8000 2100
+Wire Wire Line
+	8000 2200 8100 2200
+Text GLabel 7850 2100 0    50   Input ~ 0
 ADC-Clamp-5
 Wire Wire Line
-	7850 2000 8000 2000
-Connection ~ 8000 2000
-Wire Wire Line
-	8000 2000 8000 2100
+	7850 2100 8000 2100
+Connection ~ 8000 2100
+Wire Wire Line
+	8000 2100 8000 2200
 $Comp
 L Diode:1N5818 D5
@@
 L Diode:1N5818 D7
 U 1 1 63914F64
-P 8250 2700
-F 0 "D7" H 8250 2917 50  0000 C CNN
-F 1 "1N5818" H 8250 2826 50  0000 C CNN
-F 2 "Diode_THT:D_DO-41_SOD81_P10.16mm_Horizontal" H 8250 2525 50  0001 C CNN
-F 3 "http://www.vishay.com/docs/88525/1n5817.pdf" H 8250 2700 50  0001 C CNN
-	1    8250 2700
-	1    0    0    -1
-$EndComp
-Wire Wire Line
-	8400 2700 8500 2700
-Wire Wire Line
-	8100 2700 8000 2700
-Wire Wire Line
-	8000 2700 8000 2800
-Wire Wire Line
-	8000 2900 8100 2900
-Text GLabel 7850 2800 0    50   Input ~ 0
+P 8250 2900
+F 0 "D7" H 8250 3117 50  0000 C CNN
+F 1 "1N5818" H 8250 3026 50  0000 C CNN
+F 2 "Diode_THT:D_DO-41_SOD81_P10.16mm_Horizontal" H 8250 2725 50  0001 C CNN
+F 3 "http://www.vishay.com/docs/88525/1n5817.pdf" H 8250 2900 50  0001 C CNN
+	1    8250 2900
+	1    0    0    -1
+$EndComp
+Wire Wire Line
+	8400 2900 8500 2900
+Wire Wire Line
+	8100 2900 8000 2900
+Wire Wire Line
+	8000 2900 8000 3000
+Wire Wire Line
+	8000 3100 8100 3100
+Text GLabel 7850 3000 0    50   Input ~ 0
 ADC-Clamp-2
 Wire Wire Line
-	7850 2800 8000 2800
-Connection ~ 8000 2800
-Wire Wire Line
-	8000 2800 8000 2900
+	7850 3000 8000 3000
+Connection ~ 8000 3000
+Wire Wire Line
+	8000 3000 8000 3100
 Wire Wire Line
 	1150 6550 1150 6750
@@
 L Diode:1N5818 D12
 U 1 1 63914FDA
-P 10200 1950
-F 0 "D12" H 10200 2167 50  0000 C CNN
-F 1 "1N5818" H 10200 2076 50  0000 C CNN
-F 2 "Diode_THT:D_DO-41_SOD81_P10.16mm_Horizontal" H 10200 1775 50  0001 C CNN
-F 3 "http://www.vishay.com/docs/88525/1n5817.pdf" H 10200 1950 50  0001 C CNN
-	1    10200 1950
-	1    0    0    -1
-$EndComp
-Wire Wire Line
-	10350 1950 10450 1950
-Wire Wire Line
-	10050 1950 9950 1950
-Wire Wire Line
-	9950 1950 9950 2050
-Wire Wire Line
-	9950 2150 10050 2150
-Text GLabel 9800 2050 0    50   Input ~ 0
+P 10200 2050
+F 0 "D12" H 10200 2267 50  0000 C CNN
+F 1 "1N5818" H 10200 2176 50  0000 C CNN
+F 2 "Diode_THT:D_DO-41_SOD81_P10.16mm_Horizontal" H 10200 1875 50  0001 C CNN
+F 3 "http://www.vishay.com/docs/88525/1n5817.pdf" H 10200 2050 50  0001 C CNN
+	1    10200 2050
+	1    0    0    -1
+$EndComp
+Wire Wire Line
+	10350 2050 10450 2050
+Wire Wire Line
+	10050 2050 9950 2050
+Wire Wire Line
+	9950 2050 9950 2150
+Wire Wire Line
+	9950 2250 10050 2250
+Text GLabel 9800 2150 0    50   Input ~ 0
 ADC-Clamp-6
 Wire Wire Line
-	9800 2050 9950 2050
-Connection ~ 9950 2050
-Wire Wire Line
-	9950 2050 9950 2150
+	9800 2150 9950 2150
+Connection ~ 9950 2150
+Wire Wire Line
+	9950 2150 9950 2250
 Wire Wire Line
 	4800 1150 4950 1150
@@
 Text GLabel 10450 1150 2    50   Input ~ 0
 SigRtn
-Text GLabel 8500 2700 2    50   Input ~ 0
-SigRtn
-Text GLabel 8500 1900 2    50   Input ~ 0
+Text GLabel 8500 2900 2    50   Input ~ 0
+SigRtn
+Text GLabel 8500 2000 2    50   Input ~ 0
 SigRtn
 Text GLabel 8500 1100 2    50   Input ~ 0
 SigRtn
-Text GLabel 10450 1950 2    50   Input ~ 0
-SigRtn
-Text GLabel 10450 2750 2    50   Input ~ 0
+Text GLabel 10450 2050 2    50   Input ~ 0
+SigRtn
+Text GLabel 10450 2950 2    50   Input ~ 0
 SigRtn
 $Comp
@@
 U 1 1 6391504D
 P 8200 1300
-F 0 "D1" H 8200 1100 50  0000 C CNN
-F 1 "1N5231B" H 8200 1200 50  0000 C CNN
+F 0 "D1" H 8200 1500 50  0000 C CNN
+F 1 "1N5231B" H 8200 1400 50  0000 C CNN
 F 2 "Diode_THT:D_DO-41_SOD81_P10.16mm_Horizontal" H 8200 1300 50  0001 C CNN
 F 3 "" H 8200 1300 50  0000 C CNN
 	1    8200 1300
-	-1   0    0    -1
+	1    0    0    1
 $EndComp
 $Comp
 L V10-Ign-Inj-Drivers-V2-rescue:ZENERsmall D2
 U 1 1 63915053
-P 8200 2100
-F 0 "D2" H 8200 1900 50  0000 C CNN
-F 1 "1N5231B" H 8200 2000 50  0000 C CNN
-F 2 "Diode_THT:D_DO-41_SOD81_P10.16mm_Horizontal" H 8200 2100 50  0001 C CNN
-F 3 "" H 8200 2100 50  0000 C CNN
-	1    8200 2100
-	-1   0    0    -1
+P 8200 2200
+F 0 "D2" H 8200 2400 50  0000 C CNN
+F 1 "1N5231B" H 8200 2300 50  0000 C CNN
+F 2 "Diode_THT:D_DO-41_SOD81_P10.16mm_Horizontal" H 8200 2200 50  0001 C CNN
+F 3 "" H 8200 2200 50  0000 C CNN
+	1    8200 2200
+	1    0    0    1
 $EndComp
 $Comp
 L V10-Ign-Inj-Drivers-V2-rescue:ZENERsmall D3
 U 1 1 63915059
-P 8200 2900
-F 0 "D3" H 8200 2700 50  0000 C CNN
-F 1 "1N5231B" H 8200 2800 50  0000 C CNN
-F 2 "Diode_THT:D_DO-41_SOD81_P10.16mm_Horizontal" H 8200 2900 50  0001 C CNN
-F 3 "" H 8200 2900 50  0000 C CNN
-	1    8200 2900
-	-1   0    0    -1
+P 8200 3100
+F 0 "D3" H 8200 3300 50  0000 C CNN
+F 1 "1N5231B" H 8200 3200 50  0000 C CNN
+F 2 "Diode_THT:D_DO-41_SOD81_P10.16mm_Horizontal" H 8200 3100 50  0001 C CNN
+F 3 "" H 8200 3100 50  0000 C CNN
+	1    8200 3100
+	1    0    0    1
 $EndComp
 $Comp
@@
 U 1 1 6391505F
 P 10150 1350
-F 0 "D4" H 10150 1150 50  0000 C CNN
-F 1 "1N5231B" H 10150 1250 50  0000 C CNN
+F 0 "D4" H 10150 1550 50  0000 C CNN
+F 1 "1N5231B" H 10150 1450 50  0000 C CNN
 F 2 "Diode_THT:D_DO-41_SOD81_P10.16mm_Horizontal" H 10150 1350 50  0001 C CNN
 F 3 "" H 10150 1350 50  0000 C CNN
 	1    10150 1350
-	-1   0    0    -1
+	1    0    0    1
 $EndComp
 $Comp
 L V10-Ign-Inj-Drivers-V2-rescue:ZENERsmall D9
 U 1 1 63915065
-P 10150 2150
-F 0 "D9" H 10150 1950 50  0000 C CNN
-F 1 "1N5231B" H 10150 2050 50  0000 C CNN
-F 2 "Diode_THT:D_DO-41_SOD81_P10.16mm_Horizontal" H 10150 2150 50  0001 C CNN
-F 3 "" H 10150 2150 50  0000 C CNN
-	1    10150 2150
-	-1   0    0    -1
+P 10150 2250
+F 0 "D9" H 10150 2450 50  0000 C CNN
+F 1 "1N5231B" H 10150 2350 50  0000 C CNN
+F 2 "Diode_THT:D_DO-41_SOD81_P10.16mm_Horizontal" H 10150 2250 50  0001 C CNN
+F 3 "" H 10150 2250 50  0000 C CNN
+	1    10150 2250
+	1    0    0    1
 $EndComp
 $Comp
 L V10-Ign-Inj-Drivers-V2-rescue:ZENERsmall D10
 U 1 1 6391506B
-P 10150 2950
-F 0 "D10" H 10150 2750 50  0000 C CNN
-F 1 "1N5231B" H 10150 2850 50  0000 C CNN
-F 2 "Diode_THT:D_DO-41_SOD81_P10.16mm_Horizontal" H 10150 2950 50  0001 C CNN
-F 3 "" H 10150 2950 50  0000 C CNN
-	1    10150 2950
-	-1   0    0    -1
+P 10150 3150
+F 0 "D10" H 10150 3350 50  0000 C CNN
+F 1 "1N5231B" H 10150 3250 50  0000 C CNN
+F 2 "Diode_THT:D_DO-41_SOD81_P10.16mm_Horizontal" H 10150 3150 50  0001 C CNN
+F 3 "" H 10150 3150 50  0000 C CNN
+	1    10150 3150
+	1    0    0    1
 $EndComp
 Text GLabel 8500 1300 2    50   Input ~ 0
 SigRtn
-Text GLabel 8500 2100 2    50   Input ~ 0
-SigRtn
-Text GLabel 8500 2900 2    50   Input ~ 0
+Text GLabel 8500 2200 2    50   Input ~ 0
+SigRtn
+Text GLabel 8500 3100 2    50   Input ~ 0
 SigRtn
 Text GLabel 10450 1350 2    50   Input ~ 0
 SigRtn
-Text GLabel 10450 2150 2    50   Input ~ 0
-SigRtn
-Text GLabel 10450 2950 2    50   Input ~ 0
+Text GLabel 10450 2250 2    50   Input ~ 0
+SigRtn
+Text GLabel 10450 3150 2    50   Input ~ 0
 SigRtn
 Wire Wire Line
 	8300 1300 8500 1300
 Wire Wire Line
-	8300 2100 8500 2100
-Wire Wire Line
-	8300 2900 8500 2900
+	8300 2200 8500 2200
+Wire Wire Line
+	8300 3100 8500 3100
 Wire Wire Line
 	10250 1350 10450 1350
 Wire Wire Line
-	10250 2950 10450 2950
-Wire Wire Line
-	10250 2150 10450 2150
+	10250 3150 10450 3150
+Wire Wire Line
+	10250 2250 10450 2250
 Wire Wire Line
 	2800 3750 2650 3750
@@
 AR Path="/638ED82D/6393C9CF" Ref="D?"  Part="1"
 AR Path="/638ED685/6393C9CF" Ref="D11"  Part="1"
-F 0 "D11" H 9800 5300 50  0000 C CNN
-F 1 "1N5231B" H 9800 5200 50  0000 C CNN
+F 0 "D11" H 9800 4900 50  0000 C CNN
+F 1 "1N5231B" H 9800 5000 50  0000 C CNN
 F 2 "Diode_THT:D_DO-41_SOD81_P10.16mm_Horizontal" H 9800 5100 50  0001 C CNN
 F 3 "" H 9800 5100 50  0000 C CNN
 	1    9800 5100
-	-1   0    0    1
-$EndComp
-$Comp
+	1    0    0    -1
+$EndComp
+$Comp

Commit message: Add files via upload
Connections:
- net labels added: ADC-Clamp-0, ADC-Clamp-1, ADC-Clamp-8, MCU-A8
- net labels removed: ADC-Clamp-3, ADC-Clamp-5, ADC-Clamp-7, MCU-A7
Other:
- note added: "Spare ADC"
- note removed: "Spare ADC\n"
- moved on the sheet: D12, D9

Commit message: Add files via upload
Parts:
- removed D1, D10, D11, D2, D3, D4, D9: 1N5231B, Diode_THT:D_DO-41_SOD81_P10.16mm_Horizontal, symbol V10-Ign-Inj-Drivers-V2-rescue:ZENERsmall
- removed D12, D13, D14, D5, D6, D7, D8: 1N5818, Diode_THT:D_DO-41_SOD81_P10.16mm_Horizontal, symbol Diode:1N5818
- added J16: SP721APP, Package_DIP:DIP-8_W7.62mm, symbol Buggly~SPD:SP721APP
- added J18: Conn_01x04, Connector_PinSocket_2.54mm:PinSocket_1x04_P2.54mm_Horizontal, symbol Connector_Generic:Conn_01x04
- added R36: 1K, Resistor_THT:R_Axial_DIN0207_L6.3mm_D2.5mm_P7.62mm_Horizontal, symbol Device:R
- added R37: 2.2K, Resistor_THT:R_Axial_DIN0207_L6.3mm_D2.5mm_P7.62mm_Horizontal, symbol Device:R
Connections:
- net labels added: MCU-D0, MCU-D1
- wire segments 173 -> 140
Other:
- note added: "5V"
- note added: "ADC Clamps"
- note added: "BAT"
- note added: "BT RX"
- note added: "BT TX"
- note added: "CLT"
- note added: "DSD Tech HC-06 Bluetooth module header"
- note added: "Gnd"
- note added: "IAT"
- note added: "O2"
- note added: "RX0"
- note added: "Spare"
- note added: "TPS"
- note added: "TX0"
